File: pcb/Explorer-P.kicad_sch (KiCad schematic)
At the start: 70 parts, among them J1 GPIO Testpoint, J2 USB_C_Receptacle_USB2.0_16P, J3 RESET & BOOT, J4 TPS65-FFC0.5, J5 PWR, J6 Flash_Pin, J7 GND below MCU, J8 GPIO Testpoint, J9 GPIO Testpoint, K1 SW_Push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

Commit message: add notes on sch file
Parts:
- LD3: value Green -> Red
- R8: value 100 -> 470
Other:
- moved on the sheet: C1, C2, C5, F1, H1, H2, H3, H4, H5, H6, H7, H8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
